Commit message: update imu params

File: mavric_launch/urdf/mavric.urdf (robot description, URDF)
Before this commit: robot marvin, 15 links, 14 joints
Links:
- removed link odom
Joints:
- removed joint odom_joint

File: mavric_launch/urdf/mavric.xacro (robot description, xacro)
@@ -13,10 +13,10 @@
     </joint>
     <!-- Odom -->
-    <link name="odom" />
-    <joint name="odom_joint" type="fixed">
+    <!-- <link name="odom" />
+    <joint name="odom_joint" type="floating">
         <origin xyz="0 0 0" rpy="0 0 0" />
         <parent link="odom" />
         <child link="base_link" />
-    </joint>
+    </joint> -->
     <!-- Chassis -->
     <xacro:include filename="$(find mavric_launch)/urdf/chassis.xacro"/>
